Commit message: Fix: urdf link to data Upd: containers name set for nav

File: body/ros2/tracked_description/urdf/tracked_robot.urdf.xacro (robot description, xacro)
@@ -11,5 +11,5 @@
         <origin rpy="${rpy}" xyz="${xyz}"/>
         <geometry>
-          <mesh filename="file://$(find tracked_description)/mesh/${mesh}"
+          <mesh filename="file:///data/mesh/${mesh}"
                 scale="${scale} ${scale} ${scale}"/>
         </geometry>
@@ -18,5 +18,5 @@
         <origin rpy="${rpy}" xyz="${xyz}"/>
         <geometry>
-          <mesh filename="file://$(find tracked_description)/mesh/${mesh}"
+          <mesh filename="file:///data/mesh/${mesh}"
                 scale="${scale} ${scale} ${scale}"/>
         </geometry>
