Commit message: Upd: add woring sim

File: sim/ros2/t21_sim/config/t21.ros2_control.xacro (robot description, xacro)
@@ -13,5 +13,5 @@
       </hardware>
       <!-- виртуальный сустав линейной скорости -->
-      <joint name="left_wheel_joint">
+      <joint name="wheel_left_joint">
         <command_interface name="velocity"/>
         <state_interface   name="velocity"/>
@@ -19,5 +19,5 @@
       </joint>
       <!-- виртуальный сустав угловой скорости -->
-      <joint name="right_wheel_joint">
+      <joint name="wheel_right_joint">
         <command_interface name="velocity"/>
         <state_interface   name="velocity"/>

File: sim/ros2/t21_sim/urdf/t21.urdf.xacro (robot description, xacro)
@@ -7,5 +7,5 @@
     <!-- блок симуляции VLP-16-->
   <xacro:include filename="$(find velodyne_description)/urdf/VLP-16.urdf.xacro"/>
-  <xacro:VLP-16 parent="lidar_link"
+  <xacro:VLP-16 parent="big_box_link"
                 name="velodyne"
                 topic="/velodyne_points"
@@ -19,5 +19,5 @@
                 max_angle="3.14159265359"
                 gpu="false">
-                <origin xyz="0 0 0" rpy="0 0 0" />
+                <origin xyz="0 0 0.085" rpy="0 0 0" />
    </xacro:VLP-16>
   <xacro:include filename="$(find realsense2_description)/urdf/_d435.urdf.xacro" />

File: sim/ros2/t21_sim/urdf/tracked_robot.urdf.xacro (robot description, xacro)
@@ -178,5 +178,5 @@
   </link>
   <joint
-    name="camera_joint"
+    name="camera_base_joint"
     type="fixed">
     <origin
