Commit message: comparision test for diploma

File: src/t21_sim/urdf/imu.xacro (robot description, xacro)
@@ -53,11 +53,11 @@
           <remapping>~/out:=/imu/data_raw</remapping>
         </ros>
-        <!--topicName>imu/data_raw</topicName>
+        <!--topicName>imu/data</topicName-->
         <bodyName>xsens_link</bodyName>
         <updateRateHZ>100.0</updateRateHZ>
-        <gaussianNoise>0.001</gaussianNoise>
+        <!--gaussianNoise>0.002</gaussianNoise-->
         <xyzOffset>0 0 0</xyzOffset>
         <rpyOffset>0 0 0</rpyOffset>
-        <frameName>xsens_link</frameName-->
+        <!--frameName>xsens_link</frameName-->
       </plugin>
     </sensor>

File: src/t21_sim/urdf/t21.urdf.xacro (robot description, xacro)
@@ -19,5 +19,5 @@
                 max_angle="3.14159265359"
                 gpu="false">
-                <origin xyz="0 0 0" rpy="0 0 0" />
+                <origin xyz="0.0 0.0 0.0" rpy="0 0 0" />
    </xacro:VLP-16>
   <xacro:include filename="$(find realsense2_description)/urdf/_d435.urdf.xacro" />

File: src/t21_sim/urdf/tracked_robot.urdf.xacro (robot description, xacro)
@@ -11,4 +11,5 @@
     <color rgba="0.79216 0.81961 0.93333 1"/>
   </material>
+  <link name="lidar_link"/>
   <!-- Base Link -->
   <link name="base_link">
@@ -32,4 +33,8 @@
     </collision>
   </link>
+  <joint name="lidar_joint" type="fixed">
+    <parent link="lidar_link"/><child link="base_link"/>
+    <origin xyz="-0.1686 0.0 -0.199" rpy="0 0 0"/>
+  </joint>
   <!-- Left Wheel -->
   <link name="wheel_left_link">
@@ -178,5 +183,5 @@
   </link>
   <joint
-    name="camera_joint"
+    name="camera_base_joint"
     type="fixed">
     <origin
