Commit message: FIX: separate sim and real robot URDF descriptions

File: body/ros2/tracked_description/config/t21.ros2_control.xacro (robot description, xacro)
@@ -6,5 +6,4 @@
        несколько роботов в одном графе.
   ================================================================= -->
-  <xacro:unless value="$(arg use_sim_time)">
   <xacro:macro name="t21_ros2_control" params="name prefix">
     <ros2_control name="${name}_hw" type="system">
@@ -35,44 +34,3 @@
     <!-- Вызываем макрос, передавая имя и префикс -->
     <xacro:t21_ros2_control name="t21" prefix="$(arg prefix)"/>
-  </xacro:unless>
-  <xacro:if value="$(arg use_sim_time)">
-    <!-- ===========================================================
-       Определяем ROS 2 Control-блок для гусеничной платформы Т-21
-       Параметр prefix (по-умолчанию пустой) позволяет запускать
-       несколько роботов в одном графе.
-    ================================================================= -->
-    <ros2_control name="GazeboSystem" type="system">
-      <!-- аппаратный плагин -->
-      <hardware>
-        <plugin>gazebo_ros2_control/GazeboSystem</plugin>
-        <!-- при необходимости можно добавить <param …/> -->
-      </hardware>
-      <!-- виртуальный сустав линейной скорости -->
-      <joint name="wheel_left_joint">
-        <command_interface name="velocity"/>
-        <state_interface   name="velocity"/>
-        <state_interface name="position"/>
-      </joint>
-      <!-- виртуальный сустав угловой скорости -->
-      <joint name="wheel_right_joint">
-        <command_interface name="velocity"/>
-        <state_interface   name="velocity"/>
-        <state_interface name="position"/>
-      </joint>
-      <!--реальный сустав флиппера / стрелы -->
-      <joint name="fliper_joint">
-        <command_interface name="position"/>
-        <state_interface   name="position"/>
-      </joint>
-    </ros2_control>
-    <gazebo>
-        <plugin name="gazebo_ros2_control" filename="libgazebo_ros2_control.so">
-            <parameters>$(find t21_sim)/config/my_controllers.yaml</parameters>
-        </plugin>
-        <!-- <updateRate>10</updateRate> -->
-        <!-- <ros>
-          <remapping>odom:=odom/unfiltered</remapping>
-        </ros> -->
-    </gazebo>
-  </xacro:if>
 </robot>

File: body/ros2/tracked_description/urdf/camera.xacro (robot description, xacro)
@@ -2,5 +2,4 @@
 <robot xmlns:xacro="http://www.ros.org/wiki/xacro" >
   <xacro:property name="camera_translation" value="0.1739 0.0 0.026"/>
-  <xacro:unless value = "$(arg use_sim_time)">
     <xacro:include filename="$(find realsense2_description)/urdf/_d435.urdf.xacro"/>
     <!-- Аргументы realsense -->
@@ -12,149 +11,3 @@
       <origin xyz="${camera_translation}" rpy="0 0 0"/>
     </xacro:sensor_d435>
-  </xacro:unless>
-  <xacro:if value="$(arg use_sim_time)">
-    <xacro:arg name="depth" default="false"/>
-      <xacro:macro name="add_camera" params="name xyz">
-          <link name="${name}_link"/>
-          <joint name="${name}_joint" type="fixed">
-            <parent link="big_box_link"/>
-            <child link="${name}_link"/>
-            <origin xyz="${xyz}" rpy="0.0 -0.25 0.0"/>
-          </joint>
-          <link name="${name}_optical_link"/>
-          <joint name="${name}_optical_joint" type="fixed">
-            <parent link="${name}_link"/>
-            <child link="${name}_optical_link"/>
-            <origin xyz="0.0 0.0 0.0" rpy="${-pi/2} 0 ${-pi/2}"/>
-          </joint>
-      </xacro:macro>
-      <xacro:if value="$(arg depth)">
-          <gazebo reference="camera_link">
-              <material>Gazebo/Red</material>
-              <sensor name="camera" type="depth">
-              <pose> 0 0 0 0 0 0 </pose>
-              <visualize>true</visualize>
-              <update_rate>10</update_rate>
-              <camera>
-                  <horizontal_fov>1.089</horizontal_fov>
-                  <image>
-                      <format>B8G8R8</format>
-                      <width>640</width>
-                      <height>480</height>
-                  </image>
-                  <clip>
-                      <near>0.05</near>
-                      <far>8.0</far>
-                  </clip>
-              </camera>
-              <plugin name="camera_controller" filename="libgazebo_ros_camera.so">
-                  <!-- TODO Fix argument dependency -->
-                  <frame_name>camera_depth_optical_frame</frame_name>
-                  <min_depth>0.1</min_depth>
-                  <max_depth>100.0</max_depth>
-                  </plugin>
-              </sensor>
-          </gazebo>
-      </xacro:if>
-      <xacro:unless value="$(arg depth)">
-        <xacro:add_camera name='camera_1' xyz="${camera_translation}"/>
-        <xacro:add_camera name='camera_2' xyz="0.06 0.12 0.018"/>
-        <!-- Камера infra1 -->
-        <gazebo reference="camera_1_link">
-            <material>Gazebo/Red</material>
-            <sensor name="camera/infra1" type="camera">
-                <pose> 0.0 0.0 0.0 0 0 0 </pose>
-                <visualize>false</visualize>
-                <update_rate>10</update_rate>
-                <camera>
-                    <horizontal_fov>1.089</horizontal_fov>
-                    <image>
-                        <format>R8G8B8</format>
-                        <width>640</width>
-                        <height>480</height>
-                    </image>
-                    <clip>
-                        <near>0.05</near>
-                        <far>15.0</far>
-                    </clip>
-                </camera>
-                <plugin name="camera_controller_infra1" filename="libgazebo_ros_camera.so">
-                    <frameName>camera_1_optical_link</frameName>
-                    <cameraName>camera/infra1</cameraName>
-                    <imageTopicName>image_rect_raw</imageTopicName>
-                    <cameraInfoTopicName>camera_info</cameraInfoTopicName>
-                    <minDepth>0.1</minDepth>
-                    <maxDepth>100.0</maxDepth>
-                </plugin>
-            </sensor>
-        </gazebo>
-        <!-- Камера infra2 -->
-        <gazebo reference="camera_2_link">
-            <material>Gazebo/Orange</material>
-            <sensor name="camera/infra2" type="camera">
-                <pose> 0.0 0.0 0.0 0 0 0 </pose>  <!-- Смещение 3 см по Y для второй камеры -->
-                <visualize>false</visualize>
-                <update_rate>10</update_rate>
-                <camera>
-                    <horizontal_fov>1.089</horizontal_fov>
-                    <image>
-                        <format>R8G8B8</format>
-                        <width>640</width>
-                        <height>480</height>
-                    </image>
-                    <clip>
-                        <near>0.05</near>
-                        <far>15.0</far>
-                    </clip>
-                </camera>
-                <plugin name="camera_controller_infra2" filename="libgazebo_ros_camera.so">
-                    <frameName>camera_2_optical_link</frameName>
-                    <cameraName>camera/infra2</cameraName>
-                    <imageTopicName>image_rect_raw</imageTopicName>
-                    <cameraInfoTopicName>camera_info</cameraInfoTopicName>
-                    <minDepth>0.1</minDepth>
-                    <maxDepth>100.0</maxDepth>
-                </plugin>
-            </sensor>
-        </gazebo>
-        <link name="imu_camera_link">
-          <visual>
-            <geometry>
-              <box size="0.001 0.001 0.001"/>
-            </geometry>
-            <material name="blue">
-              <color rgba="0.0 0.0 1.0 0.5"/>
-            </material>
-          </visual>
-          <inertial>
-            <mass value="0.01"/>
-            <inertia ixx="0.00001" ixy="0.0" ixz="0.0"
-                     iyy="0.00001" iyz="0.0"
-                     izz="0.00001"/>
-          </inertial>
-        </link>
-        <joint name="imu_camera_joint" type="fixed">
-          <parent link="camera_1_link"/>
-          <child link="imu_camera_link"/>
-          <origin xyz="0.0 0.00 0.00" rpy="0 0 0"/>
-        </joint>
-        <gazebo reference="imu_camera_link">
-          <gravity>true</gravity>
-          <sensor name="imu_camera_sensor" type="imu">
-            <pose relative_to='imu_camera_link'>0 0 0 0 0 0</pose>
-            <always_on>true</always_on>
-            <update_rate>100</update_rate>
-            <plugin filename="libgazebo_ros_imu_sensor.so" name="camera_imu_plugin">
-              <ros>
-                <remapping>~/out:=/camera/imu/data</remapping>
-              </ros>
-              <frameName>imu_camera_link</frameName>
-              <topicName>camera/imu/data</topicName>
-              <bodyName>imu_camera_link</bodyName>
-              <initialOrientationAsReference>false</initialOrientationAsReference>
-            </plugin>
-          </sensor>
-        </gazebo>
-      </xacro:unless>
-  </xacro:if>
 </robot>

File: body/ros2/tracked_description/urdf/imu.xacro (robot description, xacro)
@@ -1,40 +1,6 @@
 <?xml version="1.0"?>
 <robot xmlns:xacro="http://www.ros.org/wiki/xacro">
-  <xacro:if value="$(arg use_sim_time)">
-    <!-- Макрос для инерции (добавьте в начало файла или подключите общий файл с макросами) -->
-    <xacro:macro name="box_inertia" params="b_mass b_length b_width b_height">
-      <inertial>
-        <mass value="${b_mass}"/>
-        <inertia ixx="${(b_mass/12.0) * (b_width*b_width + b_height*b_height)}"
-               ixy="0" ixz="0"
-               iyy="${(b_mass/12.0) * (b_length*b_length + b_height*b_height)}"
-               iyz="0"
-               izz="${(b_mass/12.0) * (b_length*b_length + b_width*b_width)}"/>
-      </inertial>
-    </xacro:macro>
-    <!-- Макрос геометрии IMU -->
-    <xacro:macro name="imu_link_geometry">
-      <geometry>
-        <box size="0.001 0.001 0.001"/>
-      </geometry>
-      <origin xyz="0 0 0" rpy="0 0 0"/>
-    </xacro:macro>
     <!-- Ссылка IMU -->
-    <link name="imu_link">
-      <visual>
-        <xacro:imu_link_geometry/>
-        <material name="grey">
-          <color rgba="0.5 0.5 0.5 1"/>
-        </material>
-      </visual>
-      <collision>
-        <xacro:imu_link_geometry/>
-      </collision>
-      <xacro:box_inertia
-        b_mass="0.1"
-        b_length="0.1"
-        b_width="0.1"
-        b_height="0.1"/>
-    </link>
+    <link name="imu_link"/>
     <!-- Соединение с корпусом -->
     <joint name="imu_joint" type="fixed">
@@ -43,27 +9,3 @@
       <origin xyz="0.0 0.08 0.01" rpy="0 0 0"/>
     </joint>
-    <!-- Xsense gazebo model with realistic noise and drift -->
-    <gazebo reference="imu_link">
-      <gravity>true</gravity>
-      <sensor name="imu_sensor" type="imu">
-        <pose relative_to='imu_link'>0 0 0 0 0 0</pose>
-        <always_on>true</always_on>
-        <update_rate>400</update_rate>
-        <plugin filename="libgazebo_ros_imu_sensor.so" name="imu_plugin">
-          <ros>
-            <remapping>~/out:=/imu/data</remapping>
-          </ros>
-          <!--topicName>imu/data_raw</topicName>
-          <bodyName>xsens_link</bodyName>
-          <updateRateHZ>100.0</updateRateHZ>
-          <gaussianNoise>0.001</gaussianNoise>
-          <xyzOffset>0 0 0</xyzOffset>
-          <rpyOffset>0 0 0</rpyOffset>-->
-          <frameName>imu_link</frameName>
-          <bodyName>imu_link</bodyName>
-          <initialOrientationAsReference>false</initialOrientationAsReference>
-        </plugin>
-      </sensor>
-    </gazebo>
-  </xacro:if>
 </robot>

File: body/ros2/tracked_description/urdf/lidar.xacro (robot description, xacro)
@@ -14,24 +14,3 @@
       <origin xyz="${lidar_translation}" rpy="0 0 0"/>
     </joint>
-  <!-- блок симуляции VLP-16-->
-  <xacro:if value="$(arg use_sim_time)">
-    <xacro:include filename="$(find velodyne_description)/urdf/VLP-16.urdf.xacro"/>
-    <xacro:VLP-16
-      parent="lidar_link"
-      name="velodyne"
-      topic="/velodyne_points"
-      organize_cloud="false"
-      hz="10"
-      lasers="16"
-      samples="400"
-      collision_range="0.3"
-      min_range="0.1"
-      max_range="25.0"
-      noise="0.0"
-      min_angle="-${pi}"
-      max_angle="${pi}"
-      gpu="false">
-      <origin xyz="0 0 0" rpy="0 0 0" />
-    </xacro:VLP-16>
-  </xacro:if>
 </robot>

File: body/ros2/tracked_description/urdf/t21.urdf.xacro (robot description, xacro)
@@ -3,13 +3,6 @@
   <!-- Объявляем аргументы -->
   <xacro:arg name="prefix" default=""/>
-  <!-- Использовать симуляцию -->
-  <xacro:arg name="use_sim_time" default="false"/>
   <!-- Геометрия -->
-  <xacro:unless value="$(arg use_sim_time)">
-    <xacro:include filename="$(find tracked_description)/urdf/tracked_robot.urdf.xacro"/>
-  </xacro:unless>
-  <xacro:if value="$(arg use_sim_time)">
-    <xacro:include filename="$(find t21_sim)/urdf/tracked_robot.urdf.xacro"/>
-  </xacro:if>
+  <xacro:include filename="$(find tracked_description)/urdf/tracked_robot.urdf.xacro"/>
   <!-- Блок ros2_control -->
   <xacro:include filename="$(find tracked_description)/config/t21.ros2_control.xacro"/>
